File: illuminati_rgb.kicad_sch (KiCad schematic)
At the start: 47 parts, among them IC1 TPS564247DRLR, IC2 SPH0645LM4H-1-8, J1 Conn_02x03_Odd_Even, J2 Conn_01x04, J3 Conn_01x02, J6 Conn_01x02, J7 Conn_01x04, J8 Conn_01x04, Q1 C351406, Q2 C351406, Q3 C351406, Q4 C351406, Q5 C351406, Q6 C351406, Q7 C351406, Q8 C351406, Q9 C351406, SW1 SW_SPST, U1 ESP32-WROOM-32

Commit message: v2 board
Parts:
- removed C5: 22u, Capacitor_SMD:C_0805_2012Metric, symbol Device:C
- removed IC1: TPS564247DRLR, SamacSys_Parts:SOT50P160X60-6N, symbol SamacSys_Parts:TPS564247DRLR
- removed IC2: SPH0645LM4H-1-8, SamacSys_Parts:SPH0645LM4H18, symbol SamacSys_Parts:SPH0645LM4H-1-8
- removed J2, J7, J8: Conn_01x04, TerminalBlock_Phoenix:TerminalBlock_Phoenix_MKDS-1,5-4_1x04_P5.00mm_Horizontal, symbol Connector_Generic:Conn_01x04
- removed J3, J6: Conn_01x02, TerminalBlock_Phoenix:TerminalBlock_Phoenix_MKDS-1,5-2_1x02_P5.00mm_Horizontal, symbol Connector_Generic:Conn_01x02
- removed Q1, Q2, Q3, Q4, Q5, Q6, Q7, Q8, Q9: C351406, Package_TO_SOT_SMD:SOT-23, symbol Device:Q_NMOS_GSD
- removed R10, R6, R9: 10k, Resistor_SMD:R_0805_2012Metric, symbol Device:R
- removed R11: 100k, Resistor_SMD:R_0603_1608Metric_Pad0.98x0.95mm_HandSolder, symbol Device:R
- removed R12: 22k, Resistor_SMD:R_0603_1608Metric_Pad0.98x0.95mm_HandSolder, symbol Device:R
- removed R13: NC, Resistor_SMD:R_0805_2012Metric, symbol Device:R
- removed R14: 0R, Resistor_SMD:R_0805_2012Metric, symbol Device:R
- removed R15: 10k, Resistor_SMD:R_0402_1005Metric, symbol Device:R
- removed R16: 20k, Resistor_SMD:R_0402_1005Metric, symbol Device:R
- removed SW1: SW_SPST, Button_Switch_THT:SW_PUSH_6mm_H5mm, symbol Switch:SW_SPST
- removed U1: ESP32-WROOM-32, RF_Module:ESP32-WROOM-32, symbol RF_Module:ESP32-WROOM-32
- added C1: 10u/1206, Capacitor_SMD:C_1206_3216Metric, symbol Device:C
- added C11, C12, C13, C8: 22u, Capacitor_SMD:C_0805_2012Metric, symbol Device:C
- added D1: B340A, Diode_SMD:D_SMA, symbol Device:D_Schottky
- added IC1: ESP32-C3-WROOM-02-N4, SamacSys_Parts:ESP32C3WROOM02N4, symbol SamacSys_Parts:ESP32-C3-WROOM-02-N4
- added J1: Conn_01x04, TerminalBlock_Phoenix:TerminalBlock_Phoenix_MKDS-1,5-4_1x04_P5.00mm_Horizontal, symbol Connector_Generic:Conn_01x04
- added JP1, JP2, JP3, JP4, JP5: Jumper_2_Bridged, Jumper:SolderJumper-2_P1.3mm_Bridged_RoundedPad1.0x1.5mm, symbol Jumper:Jumper_2_Bridged
- added PS1: AP5100WG-7, SamacSys_Parts:SOT95P285X140-6N, symbol SamacSys_Parts:AP5100WG-7
- added R1: 10k, Resistor_SMD:R_0603_1608Metric, symbol Device:R
- added U1: AMS1117-3.3, Package_TO_SOT_SMD:SOT-223-3_TabPin2, symbol Regulator_Linear:AMS1117-3.3
- added U2, U3, U4: 74HC14, Package_SO:SOIC-14_3.9x8.7mm_P1.27mm, symbol 74xx:74HC14
- C10: renamed from C8; value 10u -> 22u; footprint Capacitor_SMD:C_0805_2012Metric_Pad1.18x1.45mm_HandSolder -> Capacitor_SMD:C_0805_2012Metric
- C2: value 22u -> 10u/1206; footprint Capacitor_SMD:C_0805_2012Metric -> Capacitor_SMD:C_1206_3216Metric
- C3: value 100n -> 22n; footprint Capacitor_SMD:C_0603_1608Metric_Pad1.08x0.95mm_HandSolder -> Capacitor_SMD:C_0603_1608Metric
- C4, C9: value 100n -> 22u; footprint Capacitor_SMD:C_0603_1608Metric_Pad1.08x0.95mm_HandSolder -> Capacitor_SMD:C_0805_2012Metric
- C5: renamed from C1; footprint Capacitor_SMD:C_0805_2012Metric_Pad1.18x1.45mm_HandSolder -> Capacitor_SMD:C_0603_1608Metric
- C7: value 56p -> 100p; footprint Capacitor_SMD:C_0603_1608Metric_Pad1.08x0.95mm_HandSolder -> Capacitor_SMD:C_0603_1608Metric
- L1: value 1.5u -> 10u/C2921170; footprint Inductor_SMD:L_Wuerth_MAPI-4020 -> Inductor_SMD:L_Chilisin_BMRA00040420
- R2, R3, R4, R7: footprint Resistor_SMD:R_0805_2012Metric -> Resistor_SMD:R_0603_1608Metric
- R5, R8: value 10k -> 2k; footprint Resistor_SMD:R_0805_2012Metric -> Resistor_SMD:R_0603_1608Metric
- R6: renamed from R1; footprint Resistor_SMD:R_0805_2012Metric -> Resistor_SMD:R_0603_1608Metric
- renumbered J1 to J2
Connections:
- net +3V3: now also C9.1, R2.1, R3.1, IC1.1 (3V3), R1.1, U1.2 (VO); no longer C4.1, C6.1, C7.1, C9.2, L1.1
- net B1: now also IC1.5 (IO6), U2.5; no longer R8.1
- net B2: now also JP3.2 (B), U2.13
- net B3: now also IC1.13 (IO18), U3.1
- net G1: now also IC1.4 (IO5), U2.3; no longer R5.1
- net G2: now also JP5.2 (B), U2.11
- net G3: now also IC1.14 (IO19), U3.3; no longer R7.1
- net GND: now also C9.2, R5.1, C1.2, C11.2, C12.2, C13.2, C8.2, D1.2 (A), IC1.19 (GND_2), IC1.20 (GND_3), IC1.21 (GND_4), IC1.22 (GND_5), IC1.23 (GND_6), IC1.24 (GND_7), IC1.25 (GND_8), IC1.26 (GND_9), IC1.27 (GND_10), IC1.9 (GND_1), J1.3 (Pin_3), J1.4 (Pin_4), PS1.2 (GND), U1.1 (GND), U2.7 (GND), U3.7 (GND), U4.7 (GND); no longer C3.2, C9.1, R2.2, R3.2, R4.2, R5.2, R7.2
- net R1: now also IC1.3 (IO4), U2.1; no longer R2.1
- net R2: now also IC1.6 (IO7), U2.9; no longer R3.1
- net R3: now also IC1.15 (IO3), U3.5; no longer R4.1
- net VCC: now also R4.2, C1.1, J1.1 (Pin_1), J1.2 (Pin_2), PS1.5 (IN); no longer C3.1
- net boot: now also R3.2, IC1.8 (IO9), JP3.1 (A)
- net esp_en: now also IC1.2 (EN)
- net rx: now also IC1.11 (RXD), JP1.1 (A)
- net tx: now also IC1.12 (TXD), JP2.1 (A)
- net +5V: now reaches L1.2
- net +5V: now also C4.1, C6.1, C7.1, R7.1, C11.1, C12.1, C13.1, C8.1, U1.3 (VI), U2.14 (VCC), U3.14 (VCC), U4.14 (VCC)
- net V_FB: now reaches C7.2
- net V_FB: now also R7.2, R8.1, PS1.3 (FB)
- new net: C3.2, D1.1 (K), L1.1, PS1.6 (SW)
- new net: PS1.4 (EN), R4.1, R5.2
- new net: C3.1, PS1.1 (BST)
- new net B4: IC1.10 (IO10), U3.13
- new net B5: IC1.18 (IO0), U4.5
- new net G4: JP1.2 (B), U3.11
- new net G5: IC1.17 (IO1), U4.3
- new net R4: JP2.2 (B), U3.9
- new net R5: JP4.2 (B), U4.1
- new net RGB Channel1/B: U2.6
- new net RGB Channel1/G: U2.4
- new net RGB Channel1/R: U2.2
- new net RGB Channel2/B: U2.12
- new net RGB Channel2/G: U2.10
- new net RGB Channel2/R: U2.8
- new net RGB Channel3/B: U3.2
- new net RGB Channel3/G: U3.4
- new net RGB Channel3/R: U3.6
- new net RGB Channel4/B: U3.12
- new net RGB Channel4/G: U3.10
- new net RGB Channel4/R: U3.8
- new net RGB Channel5/B: U4.6
- new net RGB Channel5/G: U4.4
- new net RGB Channel5/R: U4.2
- new net gpio2: IC1.16 (IO2), JP4.1 (A), R2.2
- new net gpio8: IC1.7 (IO8), JP5.1 (A), R1.2
- no-connect marks 0 -> 6
Other:
- added sheet RGB Channel1 (rgb.kicad_sch)
- added sheet RGB Channel2 (rgb.kicad_sch)
- added sheet RGB Channel3 (rgb.kicad_sch)
- added sheet RGB Channel4 (rgb.kicad_sch)
- added sheet RGB Channel5 (rgb.kicad_sch)
- note added: "R19 = (10k * 0.81) / (Vo - 0.81)"
- moved on the sheet: C10, C5, H1, H2, J2, R6
