File: rgb.kicad_sch (KiCad schematic)
At the start: 4 parts, among them IC2 SI4174DY-T1-GE3, IC3 SI4174DY-T1-GE3, IC4 SI4174DY-T1-GE3, J1 Conn_01x04

Commit message: V2.1 swap esp32c3 for esp32 and change form factor
Parts:
- IC2, IC3, IC4: MPN (none) -> C496589
- J1: MPN (none) -> C192769
